Commit message: add cam

File: src/camera_description/urdf/camera_gazebo.xacro (robot description, xacro)
@@ -6,4 +6,5 @@
         <xacro:arg name="camera_offset_z" default="2"/>
         <!-- Create laser reference frame -->
+        <link name="world"/>
         <link name="${prefix}_link">
             <inertial>
@@ -15,5 +16,5 @@
             </inertial>
             <visual>
-                <origin xyz="$(arg camera_offset_x) $(arg camera_offset_y) $(arg camera_offset_z)" rpy="0 0 0" />
+                <origin xyz="0 0 0" rpy="0 0 0" />
                 <geometry>
                     <box size="0.01 0.04 0.04" />
@@ -29,4 +30,9 @@
             </collision>
         </link>
+       <joint name="cam_joint" type="fixed">
+            <origin xyz="$(arg camera_offset_x) $(arg camera_offset_y) $(arg camera_offset_z)" rpy="0 1.57 0"/>
+            <parent link="world"/>
+            <child link="${prefix}_link"/>
+        </joint>
         <gazebo reference="${prefix}_link">
             <material>Gazebo/Black</material>

Commit message: update camera pose

File: src/camera_description/urdf/camera_gazebo.xacro (robot description, xacro)
@@ -5,4 +5,7 @@
         <xacro:arg name="camera_offset_y" default="0"/>
         <xacro:arg name="camera_offset_z" default="2"/>
+        <xacro:arg name="row" default="0"/>
+        <xacro:arg name="pitch" default="1.57"/>
+        <xacro:arg name="yaw" default="0"/>
         <!-- Create laser reference frame -->
         <link name="world"/>
@@ -31,5 +34,5 @@
         </link>
        <joint name="cam_joint" type="fixed">
-            <origin xyz="$(arg camera_offset_x) $(arg camera_offset_y) $(arg camera_offset_z)" rpy="0 1.57 0"/>
+            <origin xyz="$(arg camera_offset_x) $(arg camera_offset_y) $(arg camera_offset_z)" rpy="$(arg row) $(arg pitch) $(arg yaw)"/>
             <parent link="world"/>
             <child link="${prefix}_link"/>
