Commit message: added beepy and tested rosbag recording

File: src/mbot_description/urdf/xacro/mbot.urdf.xacro (robot description, xacro)
@@ -33,4 +33,7 @@
     <xacro:cylinder_inertial_matrix m="1.0" r="0.05" h="0.04"/>
   </link>
+  <gazebo reference="base_link">
+            <material>Gazebo/Yellow</material>
+  </gazebo>
   <!-- Left wheel link -->
   <link name="left_wheel_link">

Commit message: update

File: src/mbot_description/urdf/xacro/mbot.urdf.xacro (robot description, xacro)
@@ -21,5 +21,5 @@
       <origin xyz="0 0 0" rpy="0 0 0"/>
       <geometry>
-        <cylinder length="0.04" radius="0.05"/>
+        <cylinder length="0.08" radius="0.05"/>
       </geometry>
       <material name="Yellow"/>
@@ -28,6 +28,12 @@
       <origin xyz="0 0 0" rpy="0 0 0"/>
       <geometry>
-        <cylinder length="0.04" radius="0.05"/>
+        <cylinder length="0.08" radius="0.05"/>
       </geometry>
+      <surface>
+        <ode>
+          <mu>1</mu>
+          <mu2>1</mu2>
+        </ode>
+      </surface>
     </collision>
     <xacro:cylinder_inertial_matrix m="1.0" r="0.05" h="0.04"/>
@@ -54,5 +60,5 @@
   </link>
   <joint name="left_wheel_joint" type="continuous">
-      <origin xyz="0 0.0475 -0.0125" rpy="0 0 0"/>
+      <origin xyz="0 0.0475 -0.0325" rpy="0 0 0"/>
       <parent link="base_link"/>
       <child link="left_wheel_link"/>
@@ -77,5 +83,5 @@
   </link>
   <joint name="right_wheel_joint" type="continuous">
-      <origin xyz="0 -0.0475 -0.0125" rpy="0 0 0"/>
+      <origin xyz="0 -0.0475 -0.0325" rpy="0 0 0"/>
       <parent link="base_link"/>
       <child link="right_wheel_link"/>
@@ -100,5 +106,5 @@
   </link>
   <joint name="front_caster_joint" type="fixed">
-      <origin xyz="0.045 0 -0.02375" rpy="0 0 0"/>
+      <origin xyz="0.045 0 -0.04375" rpy="0 0 0"/>
       <parent link="base_link"/>
       <child link="front_caster_link"/>
@@ -122,5 +128,5 @@
   </link>
   <joint name="back_caster_joint" type="fixed">
-      <origin xyz="-0.045 0 -0.02375" rpy="0 0 0"/>
+      <origin xyz="-0.045 0 -0.04375" rpy="0 0 0"/>
       <parent link="base_link"/>
       <child link="back_caster_link"/>
